File: Alt-HW/retroglowplus_gbc.kicad_pcb (KiCad board)
At the start: 2 copper layers, 78.5 x 104.2 mm, 93 parts, among them J1 MICROQTJ, Q1 BSS138DW, Q2 BSS138DW, Q3 BSS138DW, Q4 BSS138DW, SW1 1TS026A-1000-0550, U1 GD25Q80EEIGR, U2 RP2040, U3 CH9141K, U4 XC6222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

Commit message: Add gerbers
Routing:
- net GND: vias 77 -> 78
Changed lines of the file:
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@@
       (stroke (width 0.1) (type solid)) (fill solid) (layer "F.Mask"))
     (pad "1" smd custom (at -2.921 -0.9906) (size 0.75 0.75) (layers "F.Cu")
-      (net 81 "START") (pinfunction "1") (pintype "passive")
+      (net 81 "START") (pinfunction "1") (pintype "passive") (thermal_bridge_angle 45)
       (options (clearance outline) (anchor circle))
       (primitives
@@
       ))
     (pad "1" smd custom (at 0.9906 -1.0668) (size 0.75 0.75) (layers "F.Cu")
-      (net 81 "START") (pinfunction "1") (pintype "passive")
+      (net 81 "START") (pinfunction "1") (pintype "passive") (thermal_bridge_angle 45)
       (options (clearance outline) (anchor circle))
       (primitives
@@
       ))
     (pad "1" smd custom (at 2.9464 0.9906) (size 0.75 0.75) (layers "F.Cu")
-      (net 81 "START") (pinfunction "1") (pintype "passive")
+      (net 81 "START") (pinfunction "1") (pintype "passive") (thermal_bridge_angle 45)
       (options (clearance outline) (anchor circle))
       (primitives
@@
       ))
     (pad "2" smd custom (at -1.0922 -0.9906) (size 0.75 0.75) (layers "F.Cu")
-      (net 2 "GND") (pinfunction "2") (pintype "passive")
+      (net 2 "GND") (pinfunction "2") (pintype "passive") (thermal_bridge_angle 45)
       (options (clearance outline) (anchor circle))
       (primitives
@@
       ))
     (pad "2" smd custom (at 2.9718 -0.9906) (size 0.75 0.75) (layers "F.Cu")
-      (net 2 "GND") (pinfunction "2") (pintype "passive")
+      (net 2 "GND") (pinfunction "2") (pintype "passive") (thermal_bridge_angle 45)
       (options (clearance outline) (anchor circle))
       (primitives
@@
       (stroke (width 0.1) (type solid)) (layer "Dwgs.User"))
     (pad "1" smd custom (at 2.380241 -1.836461 90) (size 0.2 0.2) (layers "F.Cu")
-      (net 76 "DDOWN") (pinfunction "1") (pintype "passive")
+      (net 76 "DDOWN") (pinfunction "1") (pintype "passive") (thermal_bridge_angle 45)
       (options (clearance outline) (anchor circle))
       (primitives
@@
       ))
     (pad "2" smd custom (at 2.383405 1.820646 90) (size 0.2 0.2) (layers "F.Cu")
-      (net 2 "GND") (pinfunction "2") (pintype "passive")
+      (net 2 "GND") (pinfunction "2") (pintype "passive") (thermal_bridge_angle 45)
       (options (clearance outline) (anchor circle))
       (primitives
@@
       (stroke (width 0.1) (type solid)) (fill solid) (layer "F.Mask"))
     (pad "1" smd custom (at -2.921 -0.9906) (size 0.75 0.75) (layers "F.Cu")
-      (net 80 "SEL") (pinfunction "1") (pintype "passive")
+      (net 80 "SEL") (pinfunction "1") (pintype "passive") (thermal_bridge_angle 45)
       (options (clearance outline) (anchor circle))
       (primitives
@@
       ))
     (pad "1" smd custom (at 0.9906 -1.0668) (size 0.75 0.75) (layers "F.Cu")
-      (net 80 "SEL") (pinfunction "1") (pintype "passive")
+      (net 80 "SEL") (pinfunction "1") (pintype "passive") (thermal_bridge_angle 45)
       (options (clearance outline) (anchor circle))
       (primitives
@@
       ))
     (pad "1" smd custom (at 2.9464 0.9906) (size 0.75 0.75) (layers "F.Cu")
-      (net 80 "SEL") (pinfunction "1") (pintype "passive")
+      (net 80 "SEL") (pinfunction "1") (pintype "passive") (thermal_bridge_angle 45)
       (options (clearance outline) (anchor circle))
       (primitives
@@
       ))
     (pad "2" smd custom (at -1.0922 -0.9906) (size 0.75 0.75) (layers "F.Cu")
-      (net 2 "GND") (pinfunction "2") (pintype "passive")
+      (net 2 "GND") (pinfunction "2") (pintype "passive") (thermal_bridge_angle 45)
       (options (clearance outline) (anchor circle))
       (primitives
@@
       ))
     (pad "2" smd custom (at 2.9718 -0.9906) (size 0.75 0.75) (layers "F.Cu")
-      (net 2 "GND") (pinfunction "2") (pintype "passive")
+      (net 2 "GND") (pinfunction "2") (pintype "passive") (thermal_bridge_angle 45)
       (options (clearance outline) (anchor circle))
       (primitives
@@
       (stroke (width 0.1) (type solid)) (fill solid) (layer "F.Mask"))
     (pad "1" smd custom (at -1.1684 -2.5146) (size 0.2 0.2) (layers "F.Cu")
-      (net 66 "A") (pinfunction "1") (pintype "passive")
+      (net 66 "A") (pinfunction "1") (pintype "passive") (thermal_bridge_angle 45)
       (options (clearance outline) (anchor circle))
       (primitives
@@
       ))
     (pad "2" smd custom (at 1.155983 2.526747) (size 0.2 0.2) (layers "F.Cu")
-      (net 2 "GND") (pinfunction "2") (pintype "passive")
+      (net 2 "GND") (pinfunction "2") (pintype "passive") (thermal_bridge_angle 45)
       (options (clearance outline) (anchor circle))
       (primitives
@@
       (stroke (width 0.1) (type solid)) (layer "Dwgs.User"))
     (pad "1" smd custom (at 2.380241 -1.836461 180) (size 0.2 0.2) (layers "F.Cu")
-      (net 78 "DRIGHT") (pinfunction "1") (pintype "passive")
+      (net 78 "DRIGHT") (pinfunction "1") (pintype "passive") (thermal_bridge_angle 45)
       (options (clearance outline) (anchor circle))
       (primitives
@@
       ))
     (pad "2" smd custom (at 2.383405 1.820646 180) (size 0.2 0.2) (layers "F.Cu")
-      (net 2 "GND") (pinfunction "2") (pintype "passive")
+      (net 2 "GND") (pinfunction "2") (pintype "passive") (thermal_bridge_angle 45)
       (options (clearance outline) (anchor circle))
       (primitives
@@
       (stroke (width 0.1) (type solid)) (fill solid) (layer "F.Mask"))
     (pad "1" smd custom (at -1.1684 -2.5146) (size 0.2 0.2) (layers "F.Cu")
-      (net 75 "B") (pinfunction "1") (pintype "passive")
+      (net 75 "B") (pinfunction "1") (pintype "passive") (thermal_bridge_angle 45)
       (options (clearance outline) (anchor circle))
       (primitives
@@
       ))
     (pad "2" smd custom (at 1.155983 2.526747) (size 0.2 0.2) (layers "F.Cu")
-      (net 2 "GND") (pinfunction "2") (pintype "passive")
+      (net 2 "GND") (pinfunction "2") (pintype "passive") (thermal_bridge_angle 45)
       (options (clearance outline) (anchor circle))
       (primitives
@@
       (stroke (width 0.1) (type solid)) (layer "Dwgs.User"))
     (pad "1" smd custom (at 2.380241 -1.836461 270) (size 0.2 0.2) (layers "F.Cu")
-      (net 79 "DUP") (pinfunction "1") (pintype "passive")
+      (net 79 "DUP") (pinfunction "1") (pintype "passive") (thermal_bridge_angle 45)
       (options (clearance outline) (anchor circle))
       (primitives
@@
       ))
     (pad "2" smd custom (at 2.383405 1.820646 270) (size 0.2 0.2) (layers "F.Cu")
-      (net 2 "GND") (pinfunction "2") (pintype "passive")
+      (net 2 "GND") (pinfunction "2") (pintype "passive") (thermal_bridge_angle 45)
       (options (clearance outline) (anchor circle))
       (primitives
@@
       (stroke (width 0.1) (type solid)) (layer "Dwgs.User"))
     (pad "1" smd custom (at 2.380241 -1.836461) (size 0.2 0.2) (layers "F.Cu")
-      (net 77 "DLEFT") (pinfunction "1") (pintype "passive")
+      (net 77 "DLEFT") (pinfunction "1") (pintype "passive") (thermal_bridge_angle 45)
       (options (clearance outline) (anchor circle))
       (primitives
@@
       ))
     (pad "2" smd custom (at 2.383405 1.820646) (size 0.2 0.2) (layers "F.Cu")
-      (net 2 "GND") (pinfunction "2") (pintype "passive")
+      (net 2 "GND") (pinfunction "2") (pintype "passive") (thermal_bridge_angle 45)
       (options (clearance outline) (anchor circle))
       (primitives
@@
   (via (at 259.17 123.02) (size 0.65) (drill 0.35) (layers "F.Cu" "B.Cu") (net 2))
   (via (at 251.425 110.35) (size 0.65) (drill 0.35) (layers "F.Cu" "B.Cu") (net 2))
+  (via (at 271.0688 127.8636) (size 0.65) (drill 0.35) (layers "F.Cu" "B.Cu") (net 2))
   (via (at 247.09 134.54) (size 0.65) (drill 0.35) (layers "F.Cu" "B.Cu") (net 2))
   (via (at 272.15 124.39) (size 0.65) (drill 0.35) (layers "F.Cu" "B.Cu") (net 2))

Commit message: Update
Connections:
- R25 pad 2: BAT_IN -> BAT_LVL
- R26 pad 1: BAT_IN -> BAT_LVL
- R26 pad 2: BAT_LVL -> BAT_IN
Routing:
- net BAT_LVL: track 50.4 -> 52.7 mm
- net BAT_IN: track 47.8 -> 47.9 mm, vias 1 -> 0
Changed lines of the file:
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@@
       (net 2 "GND") (pintype "passive"))
     (pad "2" smd roundrect (at 0.32 0) (size 0.46 0.4) (layers "F.Cu" "F.Mask") (roundrect_rratio 0.25)
-      (net 8 "BAT_IN") (pintype "passive"))
+      (net 49 "BAT_LVL") (pintype "passive"))
     (model "${KICAD6_3DMODEL_DIR}/Resistor_SMD.3dshapes/R_0201_0603Metric.wrl"
       (offset (xyz 0 0 0))
@@
     (pad "" smd roundrect (at 0.345 0) (size 0.318 0.36) (layers "F.Paste") (roundrect_rratio 0.25))
     (pad "1" smd roundrect (at -0.32 0) (size 0.46 0.4) (layers "F.Cu" "F.Mask") (roundrect_rratio 0.25)
-      (net 8 "BAT_IN") (pintype "passive"))
-    (pad "2" smd roundrect (at 0.32 0) (size 0.46 0.4) (layers "F.Cu" "F.Mask") (roundrect_rratio 0.25)
       (net 49 "BAT_LVL") (pintype "passive"))
+    (pad "2" smd roundrect (at 0.32 0) (size 0.46 0.4) (layers "F.Cu" "F.Mask") (roundrect_rratio 0.25)
+      (net 8 "BAT_IN") (pintype "passive"))
     (model "${KICAD6_3DMODEL_DIR}/Resistor_SMD.3dshapes/R_0201_0603Metric.wrl"
       (offset (xyz 0 0 0))
@@
   (segment (start 237.1088 142.0136) (end 237.2888 141.8336) (width 0.25) (layer "F.Cu") (net 8))
   (segment (start 208.03 154.531) (end 208.03 145.93) (width 1) (layer "F.Cu") (net 8))
-  (segment (start 213.7 143.05) (end 214.14 143.05) (width 0.2) (layer "F.Cu") (net 8))
   (segment (start 234.9364 142.0136) (end 235.123 141.827) (width 0.6) (layer "F.Cu") (net 8))
-  (segment (start 214.139866 143.960134) (end 214.14 143.96) (width 0.2) (layer "F.Cu") (net 8))
-  (segment (start 214.14 143.05) (end 214.528 143.05) (width 0.2) (layer "F.Cu") (net 8))
+  (segment (start 214.884 143.96) (end 214.14 143.96) (width 0.2) (layer "F.Cu") (net 8))
   (segment (start 233.022 142.832) (end 234.118 142.832) (width 0.6) (layer "F.Cu") (net 8))
   (segment (start 235.123 141.2435) (end 235.1218 141.2423) (width 0.25) (layer "F.Cu") (net 8))
@@
   (segment (start 210 143.96) (end 214.14 143.96) (width 1) (layer "F.Cu") (net 8))
   (segment (start 235.123 141.2435) (end 235.123 140.66) (width 0.6) (layer "F.Cu") (net 8))
-  (segment (start 214.14 143.05) (end 214.14 143.96) (width 0.2) (layer "F.Cu") (net 8))
-  (segment (start 214.134068 143.960134) (end 214.139866 143.960134) (width 0.2) (layer "F.Cu") (net 8))
   (segment (start 208.811 154.531) (end 208.03 154.531) (width 1) (layer "F.Cu") (net 8))
   (segment (start 233.022 144.758) (end 233.022 143.795) (width 1) (layer "F.Cu") (net 8))
+  (segment (start 215.168 143.676) (end 214.884 143.96) (width 0.2) (layer "F.Cu") (net 8))
+  (segment (start 215.168 143.05) (end 215.168 143.676) (width 0.2) (layer "F.Cu") (net 8))
   (segment (start 235.123 141.827) (end 235.123 141.2435) (width 0.6) (layer "F.Cu") (net 8))
-  (via (at 214.134068 143.960134) (size 0.65) (drill 0.35) (layers "F.Cu" "B.Cu") (net 8))
   (segment (start 237.995 141.9) (end 237.929 141.834) (width 0.2) (layer "F.Cu") (net 9))
   (segment (start 237.92 139.4812) (end 237.92 139.561) (width 0.25) (layer "F.Cu") (net 9))
@@
   (segment (start 265.1 123.525) (end 263.45 123.525) (width 0.2) (layer "B.Cu") (net 47))
   (segment (start 266.3 124.725) (end 265.1 123.525) (width 0.2) (layer "B.Cu") (net 47))
+  (segment (start 213.7 143.05) (end 214.093292 143.05) (width 0.2) (layer "F.Cu") (net 49))
   (segment (start 250.091 119.172) (end 250.091 120.161) (width 0.2) (layer "F.Cu") (net 49))
-  (segment (start 222 141.71) (end 216.508 141.71) (width 0.25) (layer "F.Cu") (net 49))
+  (segment (start 214.143472 143.05) (end 214.528 143.05) (width 0.2) (layer "F.Cu") (net 49))
+  (segment (start 214.118382 143.02491) (end 214.143472 143.05) (width 0.2) (layer "F.Cu") (net 49))
+  (segment (start 214.118382 143.02491) (end 214.118382 142.319818) (width 0.25) (layer "F.Cu") (net 49))
   (segment (start 250.091 120.161) (end 250.39 120.46) (width 0.2) (layer "F.Cu") (net 49))
-  (segment (start 216.508 141.71) (end 215.168 143.05) (width 0.25) (layer "F.Cu") (net 49))
+  (segment (start 214.093292 143.05) (end 214.118382 143.02491) (width 0.2) (layer "F.Cu") (net 49))
+  (segment (start 214.118382 142.319818) (end 214.7282 141.71) (width 0.25) (layer "F.Cu") (net 49))
+  (segment (start 214.7282 141.71) (end 222 141.71) (width 0.25) (layer "F.Cu") (net 49))
   (via (at 222 141.71) (size 0.65) (drill 0.35) (layers "F.Cu" "B.Cu") (net 49))
   (via (at 250.39 120.46) (size 0.65) (drill 0.35) (layers "F.Cu" "B.Cu") (net 49))
