File: Alt-HW/retroglowplus_gbc.kicad_sch (KiCad schematic)
At the start: 83 parts, among them J1 MICROQTJ, Q1 BSS138DW, Q2 BSS138DW, Q3 BSS138DW, Q4 BSS138DW, SW1 1TS026A-1000-0550, U1 GD25Q80EEIGR, U2 RP2040, U3 CH9141K, U4 XC6222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

Commit message: Update
Connections:
- net BAT_IN: now also R26.2; no longer R25.2, R26.1
- net BAT_LVL: now also R25.2, R26.1; no longer R26.2
Changed lines of the file:
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@@
+    )
+  )
+  (global_label "BAT_IN" (shape input) (at 114.3 17.78 0) (fields_autoplaced)
+    (effects (font (size 1.27 1.27)) (justify left))
+    (property "Intersheetrefs" "${INTERSHEET_REFS}" (at 123.5143 17.78 0)
+      (effects (font (size 1.27 1.27)) (justify left) hide)
     )
   )
@@
     )
   )
-  (global_label "BAT_IN" (shape input) (at 106.68 20.32 270) (fields_autoplaced)
-    (effects (font (size 1.27 1.27)) (justify right))
-    (property "Intersheetrefs" "${INTERSHEET_REFS}" (at 106.68 29.5343 90)
-      (effects (font (size 1.27 1.27)) (justify right) hide)
-    )
-  )
   (global_label "DRIGHT" (shape input) (at 86.36 93.98 0) (fields_autoplaced)
     (effects (font (size 1.27 1.27)) (justify left))
@@
     )
   )
-  (global_label "BAT_LVL" (shape input) (at 114.3 17.78 0) (fields_autoplaced)
-    (effects (font (size 1.27 1.27)) (justify left))
-    (property "Intersheetrefs" "${INTERSHEET_REFS}" (at 124.7238 17.78 0)
-      (effects (font (size 1.27 1.27)) (justify left) hide)
-    )
-  )
   (global_label "USB_BOOT" (shape input) (at 156.21 71.12 180) (fields_autoplaced)
     (effects (font (size 1.27 1.27)) (justify right))
@@
     )
   )
+  (global_label "BAT_LVL" (shape input) (at 106.68 20.32 270) (fields_autoplaced)
+    (effects (font (size 1.27 1.27)) (justify right))
+    (property "Intersheetrefs" "${INTERSHEET_REFS}" (at 106.68 30.7438 90)
+      (effects (font (size 1.27 1.27)) (justify right) hide)
+    )
+  )
